File: DClassAmp/DClassAmp.kicad_pcb (KiCad board)
At the start: 2 copper layers, 28 parts, among them IC1 IR21834PBF, IC2 IR21834PBF, J1 ToFilterConnector, J2 PWMInputConnector, J3 MosfetGateTestpoints, J4 +12VConnector, J5 +24VConnector, Q1 IRF540N, Q2 IRF540N, Q3 IRF540N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

Commit message: Added h bridge PCB image
Routing:
- net BHO: track 63.0 -> 56.2 mm
Other:
- board text added: "A-HO"
- board text added: "A-LO"
- board text added: "B-HO"
- board text added: "B-LO"
- board text added: "ECEN405 - D Class Amp - H Bridge"
Changed lines of the file:
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@@
   (general
     (thickness 1.6)
-    (drawings 12)
-    (tracks 156)
+    (drawings 17)
+    (tracks 151)
     (zones 0)
     (modules 28)
@@
   (layers
     (0 F.Cu signal)
-    (31 B.Cu signal hide)
+    (31 B.Cu signal)
     (32 B.Adhes user)
     (33 F.Adhes user)
@@
     )
   )
+  (gr_text A-HO (at 92 83.25 90) (layer F.SilkS)
+    (effects (font (size 1 1) (thickness 0.15)))
+  )
+  (gr_text A-LO (at 90 83.25 90) (layer F.SilkS)
+    (effects (font (size 1 1) (thickness 0.15)))
+  )
+  (gr_text B-HO (at 88 83.25 90) (layer F.SilkS)
+    (effects (font (size 1 1) (thickness 0.15)))
+  )
+  (gr_text B-LO (at 86 83.25 90) (layer F.SilkS)
+    (effects (font (size 1 1) (thickness 0.15)))
+  )
+  (gr_text "ECEN405 - D Class Amp - H Bridge" (at 63 106.75 90) (layer F.SilkS)
+    (effects (font (size 1.5 1.5) (thickness 0.15)))
+  )
   (gr_text +30V (at 119 83.75) (layer F.SilkS)
     (effects (font (size 1 1) (thickness 0.15)))
@@
   (segment (start 101.01 47.75) (end 106.950001 53.690001) (width 1) (layer F.Cu) (net 19))
   (segment (start 86.87 53.08) (end 87.669999 52.280001) (width 1) (layer F.Cu) (net 19))
-  (segment (start 84.92 53.08) (end 86.87 53.08) (width 0.25) (layer F.Cu) (net 19))
-  (segment (start 84.25 53.75) (end 84.92 53.08) (width 0.25) (layer F.Cu) (net 19))
-  (segment (start 85.495001 56.745001) (end 84.25 55.5) (width 0.25) (layer F.Cu) (net 19))
-  (segment (start 84.25 55.5) (end 84.25 53.75) (width 0.25) (layer F.Cu) (net 19))
-  (segment (start 90.495001 56.745001) (end 85.495001 56.745001) (width 0.25) (layer F.Cu) (net 19))
-  (segment (start 92.5 58.75) (end 90.495001 56.745001) (width 0.25) (layer F.Cu) (net 19))
-  (segment (start 92.5 62.75) (end 92.5 58.75) (width 0.25) (layer F.Cu) (net 19))
-  (segment (start 88 67.25) (end 92.5 62.75) (width 0.25) (layer F.Cu) (net 19))
-  (segment (start 88 79.75) (end 88 67.25) (width 0.25) (layer F.Cu) (net 19))
+  (segment (start 88 79.75) (end 88 71) (width 1) (layer B.Cu) (net 19))
+  (segment (start 88 71) (end 83 66) (width 1) (layer B.Cu) (net 19))
+  (segment (start 83 66) (end 83 56.95) (width 1) (layer B.Cu) (net 19))
+  (segment (start 83 56.95) (end 86.87 53.08) (width 1) (layer B.Cu) (net 19))
   (segment (start 74.75 60.12) (end 79.25 55.62) (width 1) (layer F.Cu) (net 20))
   (segment (start 74.75 62.75) (end 74.75 60.12) (width 1) (layer F.Cu) (net 20))
