File: opFilter/pcbOutput2/pcbOutput.kicad_pcb (KiCad board)
At the start: 2 copper layers, 99.1 x 58.4 mm, 12 parts, among them J1 Conn_01x02_Female, J2 Conn_01x04_Female, J3 Conn_01x04_Female, J4 Conn_01x02_Female, J5 Conn_01x02_Female

Commit message: update
Routing:
- net Net-(J5-Pad1): track 0.00 -> 214.2 mm
- net Net-(C2-Pad1): track 0.00 -> 161.2 mm
- net Net-(C1-Pad1): track 0.00 -> 138.1 mm
- net Net-(C4-Pad2): track 0.00 -> 82.9 mm
- net Net-(J1-Pad2): track 0.00 -> 74.1 mm
- net (no net): track 0.00 -> 34.0 mm
- net GND: track 0.00 -> 12.7 mm, vias 0 -> 3
- added copper zone on B.Cu, net GND
